File: Arc/Arc.kicad_pcb (KiCad board)
At the start: 2 copper layers, 50.8 x 88.9 mm, 27 parts, among them J1 USB-C, Q1 Q_NMOS_GDS, SW1 SW_Push, T1 Transformer_1P_1S, U1 NE555D

Commit message: i forgor
Parts:
- moved J1 21.0 mm to (135.1, 124.2), turned to 0 degrees
- moved C8 12.7 mm to (135.8, 117.6), turned to 180 degrees
- moved C10 7.10 mm to (142.5, 106.9)
- moved C9 7.10 mm to (142.5, 103.9)
- moved R1 7.10 mm to (128.4, 100.3)
- moved R2 7.10 mm to (128.4, 103.3)
- moved R3 7.10 mm to (128.4, 106.2)
- moved R4 7.10 mm to (128.4, 109.2)
- moved U1 7.10 mm to (135.6, 107.2)

Commit message: Rearranging stuff
Parts:
- moved D1 23.8 mm to (150.6, 72.2), turned to 0 degrees
- moved D7 23.7 mm to (150.6, 92.3), turned to 0 degrees
- moved T1 23.2 mm to (150.2, 105.8)
- moved D2 21.3 mm to (150.6, 75.6), turned to 0 degrees
- moved D6 21.2 mm to (150.6, 89.0), turned to 0 degrees
- moved SW1 21.1 mm to (113.4, 82.5)
- moved C10 20.4 mm to (135.6, 87.6)
- moved R1 20.4 mm to (121.6, 81.1)
- moved R2 20.4 mm to (121.6, 84.0)
- moved U1 20.4 mm to (128.7, 87.9)
- moved C9 20.4 mm to (135.6, 84.6)
- moved R3 20.4 mm to (121.6, 87.0)
- moved R4 20.4 mm to (121.6, 89.9)
- moved D3 19.6 mm to (150.6, 78.9), turned to 0 degrees
- moved D5 19.6 mm to (150.6, 85.6), turned to 0 degrees
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