File: Arc/Arc.kicad_pcb (KiCad board)
At the start: 2 copper layers, 50.8 x 88.9 mm, 27 parts, among them J1 USB-C, Q1 Q_NMOS_GDS, SW1 SW_Push, T1 Transformer_1P_1S, U1 NE555D

Commit message: Finished Laser and Belle
Parts:
- added J2: Conn_01x01_Socket, Arc:5mm pad, F.Cu at (122.4, 124.6)
- added J3: Conn_01x01_Socket, Arc:5mm pad, F.Cu at (148.7, 124.5)
- added J4: Conn_01x01_Socket, Arc:5mm pad, F.Cu at (159.8, 97.5)
- added J5: Conn_01x01_Socket, Arc:5mm pad, F.Cu at (160.0, 108.6)
