File: Arc/Arc.kicad_sch (KiCad schematic)
At the start: 27 parts, among them J1 USB_C_Receptacle_PowerOnly_6P, Q1 Q_NMOS_GDS, SW1 SW_Push, T1 Transformer_1P_1S, U1 NE555D

Commit message: Adding component properties
Parts:
- C1, C2, C3, C4, C5, C6, C7: value C -> 22nF; footprint (none) -> Capacitor_SMD:C_1206_3216Metric; MPN (none) -> C1206C223KDRAC7800; Manufacturer (none) -> KEMET
- C8: value C -> 100 uF; footprint (none) -> Capacitor_SMD:C_1206_3216Metric; MPN (none) -> GRM31CD80J107MEA8K; Manufacturer (none) -> Murata Electronics
- D1, D2, D3, D4, D5, D6, D7: footprint (none) -> Diode_SMD:D_SOD-123F; MPN (none) -> 1N4007FL; Manufacturer (none) -> SMC Diode Solutions
- J1: value USB_C_Receptacle_PowerOnly_6P -> USB-C; MPN (none) -> USB4515-GF-A; Manufacturer (none) -> GCT
- Q1: footprint (none) -> Package_TO_SOT_SMD:LFPAK56; MPN (none) -> PSMN1R2-25YLC,115; Manufacturer (none) -> Nexperia USA Inc.
- T1: MPN (none) -> 53100C; Manufacturer (none) -> Murata Power Solutions Inc.
- U1: MPN (none) -> NE555DR; Manufacturer (none) -> Texas Instruments

Commit message: More component properties. PCB layout.
Need to fix component pinouts before routing.
Parts:
- C10: value C -> 10nF; footprint (none) -> Capacitor_SMD:C_0805_2012Metric; MPN (none) -> C0805C103K5RACTU; Manufacturer (none) -> KEMET
- C9: value C -> 1nF; footprint (none) -> Capacitor_SMD:C_0805_2012Metric; MPN (none) -> KGM21BCG1H102FT; Manufacturer (none) -> KYOCERA AVX
- E1: footprint (none) -> Arc:Spark Gap
- J1: footprint (none) -> Arc:GCT_USB4135-GF-A_REVA
- R1: value R_US -> 2.7k; footprint (none) -> Resistor_SMD:R_0805_2012Metric; MPN (none) -> RMCF0805FT2K70; Manufacturer (none) -> Stackpole Electronics Inc
- R2: value R_US -> 4.7k; footprint (none) -> Resistor_SMD:R_0805_2012Metric; MPN (none) -> RMCF0805FT4K70; Manufacturer (none) -> Stackpole Electronics Inc
- R3: value R_US -> 1k; footprint (none) -> Resistor_SMD:R_0805_2012Metric; MPN (none) -> RMCF0805FT1K00; Manufacturer (none) -> Stackpole Electronics Inc
- R4: value R_US -> 1M; footprint (none) -> Resistor_SMD:R_0805_2012Metric; MPN (none) -> RMCF0805FT1M00; Manufacturer (none) -> Stackpole Electronics Inc
- SW1: footprint (none) -> Arc:SW_TL3330AF260QG
- T1: footprint (none) -> Arc:53100C
Changed lines of the file:
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@@
 			)
 		)
-		(property "Value" "R_US"
+		(property "Value" "2.7k"
 			(at 124.9337 99.2252 0)
 			(effects
@@
 			)
 		)
-		(property "Footprint" ""
+		(property "Footprint" "Resistor_SMD:R_0805_2012Metric"
 			(at 123.8894 98.2093 90)
 			(effects
@@
 			)
 		)
-		(property "Datasheet" "~"
+		(property "Datasheet" "https://www.seielect.com/catalog/sei-rmcf_rmcp.pdf"
 			(at 122.8734 97.9553 0)
 			(effects
@@
 		)
 		(property "Description" "Resistor, US symbol"
+			(at 122.8734 97.9553 0)
+			(effects
+				(font
+					(size 1.27 1.27)
+				)
+				(hide yes)
+			)
+		)
+		(property "Manufacturer" "Stackpole Electronics Inc"
+			(at 122.8734 97.9553 0)
+			(effects
+				(font
+					(size 1.27 1.27)
+				)
+				(hide yes)
+			)
+		)
+		(property "MPN" "RMCF0805FT2K70"
 			(at 122.8734 97.9553 0)
 			(effects
@@
 			)
 		)
-		(property "Footprint" ""
+		(property "Footprint" "Arc:SW_TL3330AF260QG"
 			(at 97.5408 56.9239 0)
 			(effects
@@
 		(dnp no)
 		(property "Reference" "C10"
-			(at 92.773 83.7384 0)
-			(effects
-				(font
-					(size 1.27 1.27)
-				)
-			)
-		)
-		(property "Value" "C"
-			(at 95.0187 81.3644 0)
-			(effects
-				(font
-					(size 1.27 1.27)
-				)
-			)
-		)
-		(property "Footprint" ""
+			(at 94.6259 80.8995 0)
+			(effects
+				(font
+					(size 1.27 1.27)
+				)
+			)
+		)
+		(property "Value" "10nF"
+			(at 95.2705 86.3144 0)
+			(effects
+				(font
+					(size 1.27 1.27)
+				)
+			)
+		)
+		(property "Footprint" "Capacitor_SMD:C_0805_2012Metric"
 			(at 98.9353 79.7359 0)
 			(effects
@@
 			)
 		)
-		(property "Datasheet" "~"
+		(property "Datasheet" "https://content.kemet.com/datasheets/KEM_C1002_X7R_SMD.pdf"
 			(at 97.9701 83.5459 0)
 			(effects
@@
 		)
 		(property "Description" "Unpolarized capacitor"
+			(at 97.9701 83.5459 0)
+			(effects
+				(font
+					(size 1.27 1.27)
+				)
+				(hide yes)
+			)
+		)
+		(property "Manufacturer" "KEMET"
+			(at 97.9701 83.5459 0)
+			(effects
+				(font
+					(size 1.27 1.27)
+				)
+				(hide yes)
+			)
+		)
+		(property "MPN" "C0805C103K5RACTU"
 			(at 97.9701 83.5459 0)
 			(effects
@@
 			)
 		)
-		(property "Footprint" ""
+		(property "Footprint" "Arc:Spark Gap"
 			(at 252.8946 75.9577 0)
 			(effects
@@
 			)
 		)
-		(property "Footprint" ""
+		(property "Footprint" "Arc:53100C"
 			(at 153.8726 70.4799 0)
 			(effects
@@
 		(dnp no)
 		(property "Reference" "C9"
-			(at 126.2165 122.067 0)
-			(effects
-				(font
-					(size 1.27 1.27)
-				)
-			)
-		)
-		(property "Value" "C"
-			(at 127.0185 118.752 0)
-			(effects
-				(font
-					(size 1.27 1.27)
-				)
-			)
-		)
-		(property "Footprint" ""
+			(at 121.3316 117.2295 0)
+			(effects
+				(font
+					(size 1.27 1.27)
+				)
+			)
+		)
+		(property "Value" "1nF"
+			(at 121.4385 122.202 0)
+			(effects
+				(font
+					(size 1.27 1.27)
+				)
+			)
+		)
+		(property "Footprint" "Capacitor_SMD:C_0805_2012Metric"
 			(at 124.6687 115.6371 0)
 			(effects
@@
 			)
 		)
-		(property "Datasheet" "~"
+		(property "Datasheet" "https://datasheets.kyocera-avx.com/C0GNP0-KGM.pdf"
 			(at 123.7035 119.4471 0)
 			(effects
@@
 		)
 		(property "Description" "Unpolarized capacitor"
+			(at 123.7035 119.4471 0)
+			(effects
+				(font
+					(size 1.27 1.27)
+				)
+				(hide yes)
+			)
+		)
+		(property "Manufacturer" "KYOCERA AVX"
+			(at 123.7035 119.4471 0)
+			(effects
+				(font
+					(size 1.27 1.27)
+				)
+				(hide yes)
+			)
+		)
+		(property "MPN" "KGM21BCG1H102FT"
 			(at 123.7035 119.4471 0)
 			(effects
@@
 			)
 		)
-		(property "Footprint" ""
+		(property "Footprint" "Arc:GCT_USB4135-GF-A_REVA"
 			(at 44.966 70.4175 0)
 			(effects
@@
 			)
 		)
-		(property "Value" "R_US"
+		(property "Value" "1k"
 			(at 133.5825 81.5756 0)
 			(effects
@@
 			)
 		)
-		(property "Footprint" ""
+		(property "Footprint" "Resistor_SMD:R_0805_2012Metric"
 			(at 132.5382 80.5597 90)
 			(effects
@@
 			)
 		)
-		(property "Datasheet" "~"
+		(property "Datasheet" "https://www.seielect.com/catalog/sei-rmcf_rmcp.pdf"
 			(at 131.5222 80.3057 0)
 			(effects
@@
 		)
 		(property "Description" "Resistor, US symbol"
+			(at 131.5222 80.3057 0)
+			(effects
+				(font
+					(size 1.27 1.27)
+				)
+				(hide yes)
+			)
+		)
+		(property "Manufacturer" "Stackpole Electronics Inc"
+			(at 131.5222 80.3057 0)
+			(effects
+				(font
+					(size 1.27 1.27)
+				)
+				(hide yes)
+			)
+		)
+		(property "MPN" "RMCF0805FT1K00"
 			(at 131.5222 80.3057 0)
 			(effects
@@
 			)
 		)
-		(property "Value" "R_US"
+		(property "Value" "4.7k"
 			(at 125.7514 108.2179 0)
 			(effects
@@
 			)
 		)
-		(property "Footprint" ""
+		(property "Footprint" "Resistor_SMD:R_0805_2012Metric"
 			(at 124.7071 107.202 90)
 			(effects
@@
 			)
 		)
-		(property "Datasheet" "~"
+		(property "Datasheet" "https://www.seielect.com/catalog/sei-rmcf_rmcp.pdf"
 			(at 123.6911 106.948 0)
 			(effects
@@
 		)
 		(property "Description" "Resistor, US symbol"
+			(at 123.6911 106.948 0)
+			(effects
+				(font
+					(size 1.27 1.27)
+				)
+				(hide yes)
+			)
+		)
+		(property "Manufacturer" "Stackpole Electronics Inc"
+			(at 123.6911 106.948 0)
+			(effects
+				(font
+					(size 1.27 1.27)
+				)
+				(hide yes)
+			)
+		)
+		(property "MPN" "RMCF0805FT4K70"
 			(at 123.6911 106.948 0)
 			(effects
@@
 			)
 		)
-		(property "Value" "R_US"
+		(property "Value" "1M"
 			(at 136.8898 94.0116 0)
 			(effects
@@
 			)
 		)
-		(property "Footprint" ""
+		(property "Footprint" "Resistor_SMD:R_0805_2012Metric"
 			(at 135.8455 92.9957 90)
 			(effects
@@
 			)
 		)
-		(property "Datasheet" "~"
+		(property "Datasheet" "https://www.seielect.com/catalog/sei-rmcf_rmcp.pdf"
 			(at 134.8295 92.7417 0)
 			(effects
@@
 			(at 134.8295 92.7417 0)
 			(effects
+				(font
+					(size 1.27 1.27)
+				)
+				(hide yes)
+			)
+		)
+		(property "Manufacturer" "Stackpole Electronics Inc"
+			(at 134.8295 92.7417 0)
+			(effects
+				(font
+					(size 1.27 1.27)
+				)
+				(hide yes)
+			)
+		)
+		(property "MPN" "RMCF0805FT1M00"
+			(at 134.8295 92.7417 0)
+			(effects

Commit message: Finished Laser and Belle
Parts:
- added J2, J3, J4, J5: Conn_01x01_Socket, Arc:5mm pad, symbol Connector:Conn_01x01_Socket
Connections:
- net GNDREF: now also J5.1 (Pin_1)
- net at C8.2, J1.A9 (VBUS), J1.B9 (VBUS)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: now also J2.1 (Pin_1)
- net at Q1.1 (G), R3.2, R4.1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: now also J4.1 (Pin_1)
