File: Belle/Belle.kicad_pcb (KiCad board)
At the start: 2 copper layers, 43 x 33 mm, 5 parts, among them SW1 SW_Push

Commit message: Finished Laser and Belle
Parts:
- D1: footprint Belle:LED_LTW-006DCG-E2_LTO -> Belle:LED_C503D-WAN_CRW
- R1: value R_US -> 10
- SW1: moved to B.Cu
- moved R1 8.73 mm to (178.6, 109.7)
- moved SW1 8.39 mm to (188.8, 110.0), turned to -90 degrees
- moved D1 3.64 mm to (193.3, 111.3), turned to 90 degrees
- moved G*** 3.55 mm to (166.4, 109.5)
Routing:
- net Net-(BT1-+): track 0.00 -> 59.7 mm, vias 0 -> 1
- net Net-(BT1--): track 0.00 -> 36.5 mm
- net Net-(R1-Pad1): track 0.00 -> 20.5 mm, vias 0 -> 1
- net Net-(D1-A): track 0.00 -> 14.7 mm
Other:
- board size 43 x 33 mm -> 56.3 x 30.7 mm
- board text added: "etsy.com/shop/BelleBoxCo"
- board text removed: "https://www.etsy.com/shop/BelleBoxCo"
