File: Belle/Belle.kicad_sch (KiCad schematic)
At the start: 4 parts, among them SW1 SW_Push

Commit message: Finished Laser and Belle
Parts:
- D1: footprint Belle:LED_LTW-006DCG-E2_LTO -> Belle:LED_C503D-WAN_CRW; MPN LTW-006DCG-E2 -> C503D-WAN-CCBEB151; Manufacturer Lite-On Inc. -> Cree LED
Changed lines of the file:
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@@
 			)
 		)
-		(property "Footprint" "Belle:LED_LTW-006DCG-E2_LTO"
+		(property "Footprint" "Belle:LED_C503D-WAN_CRW"
 			(at 96.52 85.09 0)
 			(effects
@@
 			)
 		)
-		(property "Datasheet" "https://mm.digikey.com/Volume0/opasdata/d220001/medias/docus/379/LTW-006DCG-E2_RevH_6-12-19.pdf"
+		(property "Datasheet" "https://downloads.cree-led.com/files/ds/h/HB-C503D-WAN.pdf"
 			(at 96.52 85.09 0)
 			(effects
@@
 			)
 		)
-		(property "Manufacturer" "Lite-On Inc."
+		(property "Manufacturer" "Cree LED"
 			(at 96.52 85.09 90)
 			(effects
@@
 			)
 		)
-		(property "MPN" "LTW-006DCG-E2"
+		(property "MPN" "C503D-WAN-CCBEB151"
 			(at 96.52 85.09 90)
 			(effects
