File: Laser/Laser.kicad_pcb (KiCad board)
At the start: 2 copper layers, 50.8 x 88.9 mm, 9 parts, among them SW1 SW_Push, SW2 SW_Push, SW3 SW_Push

Commit message: Finished Laser and Belle
Parts:
- moved R1 20.4 mm to (119.2, 122.4), turned to -90 degrees
- moved R2 20.0 mm to (119.1, 117.5), turned to 180 degrees
- moved R3 9.60 mm to (131.2, 117.3)
- moved SW1 1.30 mm to (143.5, 147.5)
Routing:
- net Net-(R3-Pad2): track 0.00 -> 55.8 mm, vias 0 -> 1
- net Net-(BT1--): track 0.00 -> 50.9 mm, vias 0 -> 1
- net Net-(BT1-+): track 0.00 -> 45.9 mm
- net Net-(R1-Pad2): track 0.00 -> 40.8 mm, vias 0 -> 1
- net Net-(R2-Pad2): track 0.00 -> 40.0 mm, vias 0 -> 1
- net Net-(D1-RK): track 0.00 -> 4.42 mm
- net Net-(D1-BK): track 0.00 -> 2.52 mm
- net Net-(D1-GK): track 0.00 -> 2.35 mm
